Commit message: Just a test

File: butia_navigation_description/urdf/pioneer3at.urdf (robot description, URDF)
Before this commit: robot pioneer3at, 17 links, 16 joints
Joints:
- joint hokuyo_joint: origin xyz=0.25 0 0.31 rpy=0 0 0 -> xyz=0.25 0 0.61 rpy=0 0 0

Commit message: Created sick link based on hokuyo link files

File: butia_navigation_description/urdf/pioneer3at.urdf (robot description, URDF)
Before this commit: robot pioneer3at, 17 links, 16 joints
Links:
- added link sick_link, mass 1.1; collision box size=0.105 0.1 0.1; visual mesh filename=package://butia_navigation_description/meshes/sensors/sick_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
Joints:
- added joint sick_joint: type fixed, parent base_link, child sick_link, origin xyz=0.25 0 0.68 rpy=0 0 0
- joint hokuyo_joint: origin xyz=0.25 0 0.31 rpy=0 0 0 -> xyz=0.25 0 0.06 rpy=0 0 0

Commit message: Testing

File: butia_navigation_description/urdf/pioneer3at.urdf (robot description, URDF)
Before this commit: robot pioneer3at, 18 links, 17 joints
Joints:
- joint hokuyo_joint: origin xyz=0.25 0 0.06 rpy=3.1415 0 0 -> xyz=0.25 0 0.68 rpy=3.1415 0 0

Commit message: Testing sick parameters

File: butia_navigation_description/urdf/pioneer3at.urdf (robot description, URDF)
Before this commit: robot pioneer3at, 18 links, 17 joints
Joints:
- joint sick_joint: origin xyz=0.25 0 0.68 rpy=0 0 0 -> xyz=0.25 0 0.08 rpy=0 0 0
